File: KiCad/KeyMatrix.sch (KiCad schematic (older format))
At the start: 122 parts

Commit message: Wired Rows/Cols of Switches. Created Physical PCB.
Connections:
- net ROW5 renamed ROW4
Changed lines of the file:
@@
 ROW3
 Text GLabel 1100 4250 0    50   Input ~ 0
-ROW5
+ROW4
 Text GLabel 1750 800  1    50   Input ~ 0
 COL0
