File: KiCad/IoT_Keyboard.kicad_pcb (KiCad board)
At the start: 2 copper layers, 125 parts, among them SW1 SW_Push, U1 Elite-C

Commit message: Wired Rows/Cols of Switches. Created Physical PCB.
Parts:
- moved SW1 36.7 mm to (51.6, 84.1)
- moved R1 31.3 mm to (57.1, 83.3)
- moved U1 2.43 mm to (63.5, 68.6)
Connections:
- net ROW5 renamed ROW4
- R1 pad 1: +5V -> Net-(R1-Pad1)
- SW1 pad 1: Net-(R1-Pad2) -> Net-(R1-Pad1)
- U1 pad 21: Net-(U1-Pad21) -> Net-(R1-Pad2)
- U1 pad 22: Net-(R1-Pad2) -> Net-(R1-Pad1)
Routing:
- net ROW0: track 0.00 -> 280.7 mm
- net ROW1: track 0.00 -> 278.6 mm
- net ROW2: track 0.00 -> 271.6 mm
- net ROW4: track 0.00 -> 269.9 mm
- net ROW3: track 0.00 -> 250.0 mm
- net COL2: track 0.00 -> 89.8 mm
- net COL1: track 0.00 -> 88.9 mm
- net COL5: track 0.00 -> 83.5 mm
- net COL10: track 0.00 -> 83.4 mm
- net COL0: track 0.00 -> 83.4 mm
- net COL13: track 0.00 -> 83.3 mm
- net COL9: track 0.00 -> 82.3 mm
- net COL12: track 0.00 -> 79.3 mm
- net COL8: track 0.00 -> 64.3 mm
- net COL7: track 0.00 -> 64.3 mm
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Other:
- board outline added: 288.9 x 97.6 mm
- net class Default: trace_width 0.25 -> 0.254
- net class Power added: clearance 0.2, trace_width 0.381, via_dia 0.8, via_drill 0.4

Commit message: Routed rows and columsn to microcontroller with Daniel
 :)
Connections:
- U1 pad 10: Net-(U1-Pad10) -> COL10
- U1 pad 11: Net-(U1-Pad11) -> COL11
- U1 pad 12: Net-(U1-Pad12) -> COL12
- U1 pad 13: Net-(U1-Pad13) -> COL6
- U1 pad 14: Net-(U1-Pad14) -> COL5
- U1 pad 15: Net-(U1-Pad15) -> COL4
- U1 pad 16: Net-(U1-Pad16) -> COL3
- U1 pad 17: Net-(U1-Pad17) -> COL2
- U1 pad 18: Net-(U1-Pad18) -> COL1
- U1 pad 19: Net-(U1-Pad19) -> ROW2
- U1 pad 20: Net-(U1-Pad20) -> COL13
- U1 pad 24: Net-(U1-Pad24) -> COL0
- U1 pad 25: Net-(U1-Pad25) -> ROW4
- U1 pad 29: Net-(U1-Pad29) -> ROW3
- U1 pad 5: Net-(U1-Pad5) -> ROW0
- U1 pad 6: Net-(U1-Pad6) -> ROW1
- U1 pad 7: Net-(U1-Pad7) -> COL7
- U1 pad 8: Net-(U1-Pad8) -> COL8
- U1 pad 9: Net-(U1-Pad9) -> COL9
Routing:
- net COL13: track 83.3 -> 354.2 mm, vias 0 -> 2
- net COL12: track 79.3 -> 299.7 mm, vias 0 -> 1
- net COL11: track 42.2 -> 250.0 mm, vias 0 -> 1
- net COL10: track 83.4 -> 276.3 mm, vias 0 -> 1
- net COL9: track 82.3 -> 267.8 mm, vias 0 -> 1
- net COL8: track 64.3 -> 243.3 mm
- net COL7: track 64.3 -> 239.8 mm
- net COL6: track 64.3 -> 175.7 mm
- net COL5: track 83.5 -> 179.8 mm
- net ROW4: track 269.9 -> 350.4 mm, vias 0 -> 1
- net COL4: track 64.3 -> 144.1 mm
- net COL3: track 64.3 -> 128.8 mm
- net ROW1: track 278.6 -> 328.8 mm, vias 0 -> 3
- net COL2: track 89.8 -> 135.5 mm, vias 0 -> 1
- net ROW3: track 250.0 -> 292.4 mm, vias 0 -> 1
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
Commit message: Added HC-05 to PCB and routed. Added mounting holes. Generated gerbers
Parts:
- added R2: 1k, Resistor_SMD:R_0805_2012Metric, B.Cu at (63.9, 50.2)
- added R3: 2k, Resistor_SMD:R_0805_2012Metric, B.Cu at (63.9, 45.8)
- added REF**: MountingHole_2.2mm_M2, MountingHole:MountingHole_2.2mm_M2, F.Cu at (348.5, 41.3)
- added REF**: MountingHole_2.2mm_M2, MountingHole:MountingHole_2.2mm_M2, F.Cu at (348.5, 131.0)
- added REF**: MountingHole_2.2mm_M2, MountingHole:MountingHole_2.2mm_M2, F.Cu at (64.3, 131.0)
- added REF**: MountingHole_2.2mm_M2, MountingHole:MountingHole_2.2mm_M2, F.Cu at (64.3, 41.3)
- added U2: HC-05, Keebio:HC-05, B.Cu at (104.5, 41.0)
- moved D38 16.1 mm to (268.3, 86.5)
- moved MX38 16.1 mm to (260.4, 86.5)
- moved D17 16.1 mm to (130.2, 67.5)
- moved MX54 16.1 mm to (77.0, 124.6)
- moved R1 16.1 mm to (73.0, 81.0)
- moved D28 16.1 mm to (348.5, 66.7)
- moved D29 16.1 mm to (89.7, 86.5)
- moved D30 16.1 mm to (115.9, 86.5)
- moved D31 16.1 mm to (134.9, 86.5)
- moved D32 16.1 mm to (154.0, 86.5)
- moved D33 16.1 mm to (173.0, 86.5)
- moved D34 16.1 mm to (192.1, 86.5)
- moved D35 16.1 mm to (211.1, 86.5)
- moved D36 16.1 mm to (230.2, 86.5)
- moved D37 16.1 mm to (249.2, 86.5)
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Routing:
- net Net-(R1-Pad2): track 7.52 -> 121.3 mm, vias 0 -> 2
- net GND: track 34.2 -> 105.7 mm, vias 0 -> 1
- net Net-(U1-Pad2): track 1.78 -> 55.2 mm
- net Net-(R2-Pad1): track 0.00 -> 47.9 mm
- net COL7: track 239.8 -> 209.9 mm, vias 0 -> 4
- net COL9: track 267.8 -> 254.1 mm, vias 1 -> 2
- net COL8: track 243.3 -> 230.4 mm, vias 0 -> 4
- net Net-(R2-Pad2): track 1.78 -> 9.83 mm
- net COL11: track 250.0 -> 247.6 mm, vias 1 -> 2
- net COL0: track 113.3 -> 115.1 mm
- net COL10: track 276.3 -> 275.5 mm, vias 1 -> 2
Other:
- outline, holes or cut-outs redrawn
- board text added: "F Keys"
- board text added: "IoT Keyboard v1.0"
